File: kicad/SSDV3.kicad_pcb (KiCad board)
At the start: 4 copper layers, 58.4 x 28.8 mm, 71 parts, among them J1 SolderPad, J2 SolderPad, J3 SolderPad, J4 SolderPad, J5 SolderPad, J6 SolderPad, J7 SolderPad_01x02, J8 SolderPad_1x03, Q1 CSD19537Q3, Q2 CSD19537Q3, Q3 BSZ096N10LS5, U1 LM5050-1, U2 LM5146

Commit message: Added heatsink footprint
Parts:
- removed H1, H2, H3, H4: MountingHole, MountingHole:MountingHole_3.2mm_M3_ISO7380
- added HS1: 241802B92200G, Heatsink_JJ:24180xB9x200G, B.Cu at (149.2, 114.4)
- J7: value SolderPad_01x02 -> SolderPad_1x02
Connections:
- D5 pad 1: U2_EN -> U1_EN
- J7 pad 1: U2_EN -> U1_EN
