File: kicad/SSDV3.kicad_pcb (KiCad board)
At the start: 4 copper layers, 58.4 x 28.8 mm, 72 parts, among them J1 SolderPad, J2 SolderPad, J3 SolderPad, J4 SolderPad, J5 SolderPad, J6 SolderPad, J7 SM02B-GHS-TB(LF)(SN), J8 SM03B-GHS-TB(LF)(SN), Q1 BSZ146N10LS5, Q2 BSZ146N10LS5, Q3 BSZ146N10LS5, U1 LM5050-1, U2 LM5146

Commit message: Start of Rev E
Parts:
- removed the G*** at (147.3, 102.3)
- removed the G*** at (140.8, 107.2)
- added REF**: OMNI-UNI-34-L, Heatsink_JJ:OMNI-UNI-34-L, F.Cu at (249.0, 17.0)
- added REF**: TO-247-3_Vertical, Package_TO_SOT_THT:TO-247-3_Vertical, F.Cu at (266.9, 8.20)
- added REF**: OMNI-UNI-34-L, Heatsink_JJ:OMNI-UNI-34-L, F.Cu at (249.0, 71.0)
- added REF**: TO-247-3_Vertical, Package_TO_SOT_THT:TO-247-3_Vertical, F.Cu at (241.9, 8.20)
- added REF**: DIP-8_W7.62mm, Package_DIP:DIP-8_W7.62mm, F.Cu at (201.0, 7.50)
- added REF**: TO-247-3_Vertical, Package_TO_SOT_THT:TO-247-3_Vertical, F.Cu at (256.1, 79.8)
- added REF**: TO-247-3_Vertical, Package_TO_SOT_THT:TO-247-3_Vertical, F.Cu at (231.1, 79.8)
Other:
- board size 58.4 x 28.8 mm -> 159 x 134.8 mm
