File: kicad/SSDV3-cygnus.kicad_sch (KiCad schematic)
At the start: 8 parts, among them J3 Conn_01x02_MountingPin, J4 Conn_01x03_MountingPin

Commit message: FET Optimizations
Parts:
- removed HS1: 241802B92200G, Heatsink_JJ:24180xB9x200G, symbol Mechanical:Heatsink
- added H4, H5, H6, H7: MountingHole, MountingHole:MountingHole_3.2mm_M3_DIN965, symbol Mechanical:MountingHole
- J3: value Conn_01x02_MountingPin -> JST_GH_SM02B-GHS-TB; LCSC PN C189893 -> (none); Manufacturer JST -> (none); Part Number SM02B-GHS-TB(LF)(SN) -> (none); Part Type Extended -> (none)
- J4: value Conn_01x03_MountingPin -> JST_GH_SM03B-GHS-TB; LCSC PN C514175 -> (none); Manufacturer JST -> (none); Part Number SM03B-GHS-TB(LF)(SN) -> (none); Part Type Extended -> (none)
- renumbered D4 to D5, D3 to D6
Connections:
- net PGND: no longer J3.MP (MountPin), J4.MP (MountPin)
- no-connect marks 0 -> 2
