File: kicad/SSDV3.kicad_sch (KiCad schematic)
At the start: 8 parts, among them J3 Conn_01x02_MountingPin, J4 Conn_01x03_MountingPin

Commit message: Wrong design files initially commited
Parts:
- removed J3: Conn_01x02_MountingPin, Connector_JST:JST_GH_SM02B-GHS-TB_1x02-1MP_P1.25mm_Horizontal, symbol Connector_Generic_MountingPin:Conn_01x02_MountingPin
- removed J4: Conn_01x03_MountingPin, Connector_JST:JST_GH_SM03B-GHS-TB_1x03-1MP_P1.25mm_Horizontal, symbol Connector_Generic_MountingPin:Conn_01x03_MountingPin
- added J7: SM02B-GHS-TB(LF)(SN), Connector_JST:JST_GH_SM02B-GHS-TB_1x02-1MP_P1.25mm_Horizontal, symbol Connector_Generic_MountingPin:Conn_01x02_MountingPin
- added J8: SM03B-GHS-TB(LF)(SN), Connector_JST:JST_GH_SM03B-GHS-TB_1x03-1MP_P1.25mm_Horizontal, symbol Connector_Generic_MountingPin:Conn_01x03_MountingPin
- renumbered D4 to D5, D3 to D6
Connections:
- net PG: now also J8.2 (Pin_2)
- net PGND: now also J7.2 (Pin_2), J7.MP (MountPin), J8.3 (Pin_3), J8.MP (MountPin)
- net VCC: now also J8.1 (Pin_1)
- net U1_EN renamed U2_EN
- net U2_EN: now also J7.1 (Pin_1)
Other:
- added sheet rpp (rpp.kicad_sch)
