File: kicad/SSDV3.kicad_sch (KiCad schematic)
At the start: 8 parts, among them J7 SM02B-GHS-TB(LF)(SN), J8 SM03B-GHS-TB(LF)(SN)

Commit message: Start of Rev E
Parts:
- D5, D6, J8: Hand Assembled (none) -> N
- J7: Hand Assembled (none) -> Y
