File: kicad/buck_converter.kicad_sch (KiCad schematic)
At the start: 47 parts, among them J5 SolderPad, J6 SolderPad, Q2 BSZ146N10LS5, Q3 BSZ146N10LS5, U2 LM5146

Commit message: Start of Rev E
Parts:
- removed Q2, Q3: BSZ146N10LS5, Package_SON_JJ:Infineon_PG-TSDSON-8-26_3.3x3.3mm_P0.65mm_ThermalVias-D0.3mm, symbol Julian_Symbols:BSZ096N10LS5
- added Q2, Q3: NTMFS015N10MCL, Package_SON_JJ:Onsemi_DFN-5-EP_6x5mm_P1.27mm, symbol Transistor_FET:FDMS86150
- C10, C11, C12, C13, C14, C15, C16, C17, C4, C5, C6, C7, C8, C9, D4, R10, R11, R12, R13, R14, R15, R17, R2, R3, R4, R6, R8, R9, U2: Hand Assembled (none) -> N
- C18, C19, C20, C21, C22, C23, C24, L1, R16: Hand Assembled (none) -> Y
- R5: value 24k -> 47k; Hand Assembled (none) -> N; LCSC PN C23352 -> C25819; Part Number 0603WAF2402T5E -> 0603WAF4702T5E
Connections:
- net HO: now also Q2.4 (G)
- net LO: now also Q3.4 (G)
- net PGND: now also Q3.1 (S), Q3.2 (S), Q3.3 (S)
- net SW: now also Q2.1 (S), Q2.2 (S), Q2.3 (S), Q3.5 (D)
- net VIN: now also Q2.5 (D)
Other:
- note added: "f_{SW} = 212kHz"
- note removed: "f_{SW} = 420kHz"
