File: kicad/rpp.kicad_sch (KiCad schematic)
At the start: 13 parts, among them J1 SolderPad, J2 SolderPad, J3 SolderPad, J4 SolderPad, Q1 BSZ146N10LS5, U1 LM5050-1

Commit message: Start of Rev E
Parts:
- C1: Hand Assembled (none) -> Y
- C2, C3, D1, D2, D3, Q1, R1, U1: Hand Assembled (none) -> N
